File: MCU.kicad_sch (KiCad schematic)
At the start: 23 parts, among them J4 Conn_01x04, J5 FLAT za displej, U7 STM32F103C8Tx, Y1 32.768K, Y2 8MHz

Commit message: Postavljen je Switch na šematiku za mikrokontroler, takođe je povezan na PCB-u.
Parts:
- added SW1: SW_Push, Button_Switch_SMD:SW_Tactile_SPST_NO_Straight_CK_PTS636Sx25SMTRLFS, symbol Switch:SW_Push
Connections:
- net GND: now also SW1.1
- net RST: now also SW1.2
Changed lines of the file:
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@@
   (junction (at 237.49 32.385) (diameter 0) (color 0 0 0 0)
+  )
+  (junction (at 46.355 48.26) (diameter 0) (color 0 0 0 0)
   )
   (junction (at 255.27 32.385) (diameter 0) (color 0 0 0 0)
@@
     (stroke (width 0) (type default) (color 0 0 0 0))
   )
+  (wire (pts (xy 40.64 37.465) (xy 46.355 37.465))
+    (stroke (width 0) (type default) (color 0 0 0 0))
+  )
   (wire (pts (xy 42.545 67.31) (xy 42.545 66.04))
     (stroke (width 0) (type default) (color 0 0 0 0))
@@
     (stroke (width 0) (type default) (color 0 0 0 0))
   )
+  (wire (pts (xy 30.48 37.465) (xy 30.48 48.26))
+    (stroke (width 0) (type default) (color 0 0 0 0))
+  )
   (wire (pts (xy 52.07 37.465) (xy 46.355 37.465))
     (stroke (width 0) (type default) (color 0 0 0 0))
@@
   )
   (wire (pts (xy 25.4 57.15) (xy 20.955 57.15))
+    (stroke (width 0) (type default) (color 0 0 0 0))
+  )
+  (wire (pts (xy 30.48 48.26) (xy 46.355 48.26))
     (stroke (width 0) (type default) (color 0 0 0 0))
   )
@@
     (pin "1")
   )
+  (symbol (lib_id "Switch:SW_Push") (at 35.56 37.465 0) (unit 1)
+    (in_bom yes) (on_board yes) (fields_autoplaced)
+    (property "Reference" "SW1" (id 0) (at 35.56 29.21 0))
+    (property "Value" "SW_Push" (id 1) (at 35.56 31.75 0))
+    (property "Footprint" "Button_Switch_SMD:SW_Tactile_SPST_NO_Straight_CK_PTS636Sx25SMTRLFS" (id 2) (at 35.56 32.385 0)
+      (effects (font (size 1.27 1.27)) hide)
+    )
+    (property "Datasheet" "~" (id 3) (at 35.56 32.385 0)
+      (effects (font (size 1.27 1.27)) hide)
+    )
+    (pin "1")
+    (pin "2")
+  )
   (symbol (lib_id "power:GND") (at 106.045 62.865 0) (unit 1)
